File: iteration1_pcbs/iteration1_pcb/igniter_actuator.sch (KiCad schematic (older format))
At the start: 39 parts

Commit message: Reorganising pcb folders and adding test pcb
Connections:
- net 48V: no longer J?.1 (Pin_1), J?.1 (Pin_1)
- net CAP_HIGH: now also J?.1 (Pin_1), J?.1 (Pin_1)
Other:
- moved on the sheet: J?
Changed lines of the file:
@@
 L Connector:Screw_Terminal_01x01 J?
 U 1 1 60D67510
-P 9400 4625
-F 0 "J?" H 9480 4667 50  0000 L CNN
-F 1 "FET_A_P" H 9480 4576 50  0000 L CNN
-F 2 "" H 9400 4625 50  0001 C CNN
-F 3 "~" H 9400 4625 50  0001 C CNN
-	1    9400 4625
+P 9725 4625
+F 0 "J?" H 9805 4667 50  0000 L CNN
+F 1 "FET_A_P" H 9805 4576 50  0000 L CNN
+F 2 "" H 9725 4625 50  0001 C CNN
+F 3 "~" H 9725 4625 50  0001 C CNN
+	1    9725 4625
 	1    0    0    -1
 $EndComp
@@
 L Connector:Screw_Terminal_01x01 J?
 U 1 1 60D6902C
-P 9400 4900
-F 0 "J?" H 9480 4942 50  0000 L CNN
-F 1 "FET_A_N" H 9480 4851 50  0000 L CNN
-F 2 "" H 9400 4900 50  0001 C CNN
-F 3 "~" H 9400 4900 50  0001 C CNN
-	1    9400 4900
+P 9725 4900
+F 0 "J?" H 9805 4942 50  0000 L CNN
+F 1 "FET_A_N" H 9805 4851 50  0000 L CNN
+F 2 "" H 9725 4900 50  0001 C CNN
+F 3 "~" H 9725 4900 50  0001 C CNN
+	1    9725 4900
 	1    0    0    -1
 $EndComp
@@
 L Connector:Screw_Terminal_01x01 J?
 U 1 1 60D695B2
-P 9400 5175
-F 0 "J?" H 9480 5217 50  0000 L CNN
-F 1 "FET_B_P" H 9480 5126 50  0000 L CNN
-F 2 "" H 9400 5175 50  0001 C CNN
-F 3 "~" H 9400 5175 50  0001 C CNN
-	1    9400 5175
+P 9725 5175
+F 0 "J?" H 9805 5217 50  0000 L CNN
+F 1 "FET_B_P" H 9805 5126 50  0000 L CNN
+F 2 "" H 9725 5175 50  0001 C CNN
+F 3 "~" H 9725 5175 50  0001 C CNN
+	1    9725 5175
 	1    0    0    -1
 $EndComp
@@
 L Connector:Screw_Terminal_01x01 J?
 U 1 1 60D69B42
-P 9400 5450
-F 0 "J?" H 9480 5492 50  0000 L CNN
-F 1 "FET_B_N" H 9480 5401 50  0000 L CNN
-F 2 "" H 9400 5450 50  0001 C CNN
-F 3 "~" H 9400 5450 50  0001 C CNN
-	1    9400 5450
+P 9725 5450
+F 0 "J?" H 9805 5492 50  0000 L CNN
+F 1 "FET_B_N" H 9805 5401 50  0000 L CNN
+F 2 "" H 9725 5450 50  0001 C CNN
+F 3 "~" H 9725 5450 50  0001 C CNN
+	1    9725 5450
 	1    0    0    -1
 $EndComp
-Text Label 9200 4900 2    50   ~ 0
+Text Label 9525 4900 2    50   ~ 0
 FET_A
-Text Label 9200 5450 2    50   ~ 0
+Text Label 9525 5450 2    50   ~ 0
 FET_B
-Text Label 9200 4625 2    50   ~ 0
-48V
-Text Label 9200 5175 2    50   ~ 0
-48V
+Text Label 9525 4625 2    50   ~ 0
+CAP_HIGH
+Text Label 9525 5175 2    50   ~ 0
+CAP_HIGH
 Text HLabel 1625 5400 0    50   Input ~ 0
 CAP_DCHG
