File: iteration1_pcbs/iteration1_pcb/iteration1.sch (KiCad schematic (older format))
At the start: 24 parts

Commit message: Reorganising pcb folders and adding test pcb
Parts:
- added J?: AYF531235, CONN_AYF531235_PAN, symbol symbols:AYF531235
Connections:
- net CTS1: now also J?.3
- net GND: now also J?.6, J?.7
- net RTS1: now also J?.4
- net RX1: now also J?.1
- net RX2: now also J?.12
- net SCL1: now also J?.9
- net SDA1: now also J?.10
- net TX1: now also J?.2
- net TX2: now also J?.11
- net VCC: now also J?.5, J?.8
Other:
- note added: "GPS and Telemetry Flat Flex"
Changed lines of the file:
@@
 Text Label 3600 4050 0    50   ~ 0
 CAP_SENSE
-Text Label 7975 3150 2    50   ~ 0
+Text Label 9900 4200 2    50   ~ 0
 RX1
-Text Label 7975 3250 2    50   ~ 0
+Text Label 9900 4300 2    50   ~ 0
 TX1
-Text Label 7975 3350 2    50   ~ 0
+Text Label 9900 4400 2    50   ~ 0
 CTS1
-Text Label 7975 3450 2    50   ~ 0
+Text Label 9900 4500 2    50   ~ 0
 RTS1
-Text Label 7975 3675 2    50   ~ 0
+Text Label 9900 5300 2    50   ~ 0
 RX2
-Text Label 7975 3775 2    50   ~ 0
+Text Label 9900 5200 2    50   ~ 0
 TX2
-Text Label 7975 3975 2    50   ~ 0
+Text Label 9900 5100 2    50   ~ 0
 SDA1
-Text Label 7975 3875 2    50   ~ 0
+Text Label 9900 5000 2    50   ~ 0
 SCL1
 $Comp
@@
 L power:GND #PWR?
 U 1 1 60E50C93
-P 7675 3600
-F 0 "#PWR?" H 7675 3350 50  0001 C CNN
-F 1 "GND" H 7680 3427 50  0000 C CNN
-F 2 "" H 7675 3600 50  0001 C CNN
-F 3 "" H 7675 3600 50  0001 C CNN
-	1    7675 3600
+P 9700 4700
+F 0 "#PWR?" H 9700 4450 50  0001 C CNN
+F 1 "GND" H 9705 4527 50  0000 C CNN
+F 2 "" H 9700 4700 50  0001 C CNN
+F 3 "" H 9700 4700 50  0001 C CNN
+	1    9700 4700
 	1    0    0    -1
 $EndComp
@@
 L power:VCC #PWR?
 U 1 1 60E63803
-P 7675 3475
-F 0 "#PWR?" H 7675 3325 50  0001 C CNN
-F 1 "VCC" H 7690 3648 50  0000 C CNN
-F 2 "" H 7675 3475 50  0001 C CNN
-F 3 "" H 7675 3475 50  0001 C CNN
-	1    7675 3475
+P 9550 4600
+F 0 "#PWR?" H 9550 4450 50  0001 C CNN
+F 1 "VCC" H 9565 4773 50  0000 C CNN
+F 2 "" H 9550 4600 50  0001 C CNN
+F 3 "" H 9550 4600 50  0001 C CNN
+	1    9550 4600
 	1    0    0    -1
 $EndComp
+$Comp
+L symbols:AYF531235 J?
+U 1 1 60E7C415
+P 9900 4200
+F 0 "J?" H 10428 3703 60  0000 L CNN
+F 1 "AYF531235" H 10428 3597 60  0000 L CNN
+F 2 "CONN_AYF531235_PAN" H 10175 4365 60  0001 C CNN
+F 3 "" H 9900 4200 60  0000 C CNN
+	1    9900 4200
+	1    0    0    -1
+$EndComp
+Wire Wire Line
+	9550 4600 9900 4600
+Wire Wire Line
+	9700 4700 9900 4700
+Wire Wire Line
+	9900 4700 9900 4800
+Connection ~ 9900 4700
+Wire Wire Line
+	9550 4600 9550 4900
+Wire Wire Line
+	9550 4900 9900 4900
+Connection ~ 9550 4600
+Text Notes 9575 5600 0    50   ~ 0
+GPS and Telemetry Flat Flex
 $EndSCHEMATC

Commit message: Starting the igniter pcb
Other:
- moved on the sheet: TH?
Changed lines of the file:
@@
 L Device:Thermistor_NTC TH?
 U 1 1 60DE089F
-P 9675 3475
-F 0 "TH?" H 9773 3521 50  0000 L CNN
-F 1 "SL05 4R003" H 9773 3430 50  0000 L CNN
-F 2 "" H 9675 3525 50  0001 C CNN
-F 3 "~" H 9675 3525 50  0001 C CNN
-	1    9675 3475
+P 9225 3400
+F 0 "TH?" H 9323 3446 50  0000 L CNN
+F 1 "SL05 4R003" H 9323 3355 50  0000 L CNN
+F 2 "" H 9225 3450 50  0001 C CNN
+F 3 "~" H 9225 3450 50  0001 C CNN
+	1    9225 3400
 	1    0    0    -1
 $EndComp
@@
 L power:VCC #PWR?
 U 1 1 60DE63D3
-P 9675 3250
-F 0 "#PWR?" H 9675 3100 50  0001 C CNN
-F 1 "VCC" H 9690 3423 50  0000 C CNN
-F 2 "" H 9675 3250 50  0001 C CNN
-F 3 "" H 9675 3250 50  0001 C CNN
-	1    9675 3250
-	1    0    0    -1
-$EndComp
-Wire Wire Line
-	9675 3250 9675 3325
-Text Label 9675 3725 0    50   ~ 0
+P 9225 3175
+F 0 "#PWR?" H 9225 3025 50  0001 C CNN
+F 1 "VCC" H 9240 3348 50  0000 C CNN
+F 2 "" H 9225 3175 50  0001 C CNN
+F 3 "" H 9225 3175 50  0001 C CNN
+	1    9225 3175
+	1    0    0    -1
+$EndComp
+Wire Wire Line
+	9225 3175 9225 3250
+Text Label 9225 3650 0    50   ~ 0
 VBAT
 Wire Wire Line
-	9675 3725 9675 3625
+	9225 3650 9225 3550
 $Comp
 L Connector_Generic:Conn_01x02 J?
@@
 Text Label 10175 3225 2    50   ~ 0
 VBAT
-Text Label 10175 3325 2    50   ~ 0
-GND
 $Comp
 L symbols:HFW8R-1STE1H1LF J?
@@
 Text Notes 9575 5600 0    50   ~ 0
 GPS and Telemetry Flat Flex
+$Comp
+L power:GND #PWR?
+U 1 1 60EAC52B
+P 10050 3325
+F 0 "#PWR?" H 10050 3075 50  0001 C CNN
+F 1 "GND" H 10055 3152 50  0000 C CNN
+F 2 "" H 10050 3325 50  0001 C CNN
+F 3 "" H 10050 3325 50  0001 C CNN
+	1    10050 3325
+	1    0    0    -1
+$EndComp
+Wire Wire Line
+	10050 3325 10175 3325
 $EndSCHEMATC
